Commit message: 替换为了官方usd

File: assets/robots/holosoma_g1/g1_29dof.urdf (robot description, URDF)
Before this commit: robot g1, 42 links, 41 joints
Links:
- removed link left_sphere_hand_link
- removed link right_sphere_hand_link
- added link left_rubber_hand, mass 0.170; visual mesh filename=meshes/left_rubber_hand.STL
- added link right_rubber_hand, mass 0.170; visual mesh filename=meshes/right_rubber_hand.STL
- link LL_FOOT: geometry visual box size=0.001 0.001 0.001
- link LR_FOOT: geometry visual box size=0.001 0.001 0.001
- link head_link: geometry visual mesh filename=meshes/head_link.STL
- link imu_in_pelvis: geometry visual box size=0.001 0.001 0.001
- link imu_in_torso: geometry visual box size=0.001 0.001 0.001
- link left_elbow_link: geometry collision cylinder length=0.13 radius=0.035; visual mesh filename=meshes/left_elbow_link.STL
- link left_foot_contact_point: geometry visual box size=0.001 0.001 0.001
- link left_hip_roll_link: geometry collision cylinder length=0.2 radius=0.05; visual mesh filename=meshes/left_hip_roll_link.STL
- link left_hip_yaw_link: geometry visual mesh filename=meshes/left_hip_yaw_link.STL
- link left_wrist_pitch_link: geometry visual mesh filename=meshes/left_wrist_pitch_link.STL
- link left_wrist_roll_link: geometry visual mesh filename=meshes/left_wrist_roll_link.STL
- link left_wrist_yaw_link: geometry collision cylinder length=0.05 radius=0.05; visual mesh filename=meshes/left_wrist_yaw_link.STL
- link mid360_link: geometry visual box size=0.001 0.001 0.001
- link right_elbow_link: geometry collision cylinder length=0.13 radius=0.035; visual mesh filename=meshes/right_elbow_link.STL
- link right_foot_contact_point: geometry visual box size=0.001 0.001 0.001
- link right_hip_roll_link: geometry collision cylinder length=0.2 radius=0.05; visual mesh filename=meshes/right_hip_roll_link.STL
- link right_hip_yaw_link: geometry visual mesh filename=meshes/right_hip_yaw_link.STL
- link right_wrist_pitch_link: geometry visual mesh filename=meshes/right_wrist_pitch_link.STL
- link right_wrist_roll_link: geometry visual mesh filename=meshes/right_wrist_roll_link.STL
- link right_wrist_yaw_link: geometry collision cylinder length=0.05 radius=0.05; visual mesh filename=meshes/right_wrist_yaw_link.STL
- link torso_link: geometry collision cylinder length=0.01 radius=0.068; collision cylinder length=0.04 radius=0.065
Joints:
- joint left_hand_palm_joint: child left_sphere_hand_link -> left_rubber_hand; origin xyz=0.029 -0.003 0 rpy=0 1.57 0 -> xyz=0.0415 0.003 0 rpy=0 0 0
- joint right_hand_palm_joint: child right_sphere_hand_link -> right_rubber_hand; origin xyz=0.029 -0.003 0 rpy=0 1.57 0 -> xyz=0.0415 -0.003 0 rpy=0 0 0
